File: power_supply.kicad_sch (KiCad schematic)
At the start: 18 parts, among them Q1 2N3904, U1 LM2596S-5, U2 AMS1117-5.0

Commit message: finished without LAN
Parts:
- removed C1: EEHZA1V151P, footprints:CAP_EEHZA1V151P, symbol EEHZA1V151P:EEHZA1V151P
- removed C2: EMVH350GDA331MLH0S, footprints:CAP_EMVH630GDA331MLH0S, symbol Device:C_Polarized_US
- removed C3: 10u, Capacitor_SMD:C_1206_3216Metric_Pad1.33x1.80mm_HandSolder, symbol Device:C_Polarized
- removed C4: 22u, Capacitor_SMD:C_1206_3216Metric_Pad1.33x1.80mm_HandSolder, symbol Device:C_Polarized
- removed D1: B560C-13-F, digikey-footprints:DO-214AB, symbol dk_Diodes-Rectifiers-Single:B560C-13-F
- removed D2: MBR230LSFT1G, footprints:SODFL3616X98N, symbol Device:D_Schottky
- removed D3: SMCJ26CA-13-F, footprints:DIOM7959X250N, symbol Device:D_TVS
- removed D5: MMBZ5240BLT1G, footprints:SOT96P237X111-3N, symbol Device:D_Zener_Filled
- removed F1: MF-USHT050KX-2, footprints:FUSC3226X85N, symbol Device:Polyfuse
- removed L1: IHLP6767DZER470M11, footprints:IHLP6767DZER470M11, symbol IHLP6767DZER470M11:IHLP6767DZER470M11
- removed Q1: 2N3904, digikey-footprints:TO-92-3, symbol dk_Transistors-Bipolar-BJT-Single:2N3904
- removed U1: LM2596S-5, Package_TO_SOT_SMD:TO-263-5_TabPin3, symbol Regulator_Switching:LM2596S-5
- removed U2: AMS1117-5.0, Package_TO_SOT_SMD:SOT-223-3_TabPin2, symbol Regulator_Linear:AMS1117-5.0
- added C1: 10n, Capacitor_SMD:C_0603_1608Metric_Pad1.08x0.95mm_HandSolder, symbol Device:C
- added C10, C3, C4, C9: 22u, Capacitor_SMD:C_1206_3216Metric_Pad1.33x1.80mm_HandSolder, symbol Device:C
- added C11, C14, C8: 100n, Capacitor_SMD:C_0603_1608Metric_Pad1.08x0.95mm_HandSolder, symbol Device:C
- added C2, C7: 10u, Capacitor_SMD:C_1206_3216Metric_Pad1.33x1.80mm_HandSolder, symbol Device:C
- added D2: SMCJ26CA, footprints:DIONM7959X262N, symbol SMCJ26CA:SMCJ26CA
- added D4: D_Schottky, footprints:SOD2513X120N, symbol Device:D_Schottky
- added F2: Polyfuse, footprints:FUSC3226X85N, symbol Device:Polyfuse
- added IC1: TPS563300DRLR, footprints:TPS62932DRLR, symbol TPS563300DRLR:TPS563300DRLR
- added IC2: MMSZ5231BS-7-F, footprints:SOD2513X120N, symbol MMSZ5231BS-7-F:MMSZ5231BS-7-F
- added L1: 6.8uH, footprints:74439346068, symbol Device:L
- added R4: 49.9k, Resistor_SMD:R_0603_1608Metric_Pad0.98x0.95mm_HandSolder, symbol Device:R
- added R5: 49.9, Resistor_SMD:R_0603_1608Metric_Pad0.98x0.95mm_HandSolder, symbol Device:R
- added R8: 0, Resistor_SMD:R_0603_1608Metric_Pad0.98x0.95mm_HandSolder, symbol Device:R
- added TP4, TP5, TP6, TP7, TP8: (no value), TestPoint:TestPoint_Pad_1.5x1.5mm, symbol Connector:TestPoint_Small
- added U1: AMS1117-3.3, Package_TO_SOT_SMD:SOT-223-3_TabPin2, symbol Regulator_Linear:AMS1117-3.3
- C5, C6: footprint Capacitor_SMD:C_1206_3216Metric_Pad1.33x1.80mm_HandSolder -> Capacitor_SMD:C_0603_1608Metric_Pad1.08x0.95mm_HandSolder; JLCPCB Part # (none) -> C519438; part number (none) -> CC0603KRX7R6BB104
- R1: value 10k -> 53.6k; footprint Resistor_SMD:R_1206_3216Metric_Pad1.30x1.75mm_HandSolder -> Resistor_SMD:R_0603_1608Metric_Pad0.98x0.95mm_HandSolder; JLCPCB Part # (none) -> C137700; part number (none) -> RC0603FR-0753K6L
- R2: value 10k -> 10.2k; footprint Resistor_SMD:R_1206_3216Metric_Pad1.30x1.75mm_HandSolder -> Resistor_SMD:R_0603_1608Metric_Pad0.98x0.95mm_HandSolder; JLCPCB Part # (none) -> C183219; part number (none) -> RC0603FR-0710K2L
- R3: value 47k -> 49.9k; footprint Resistor_SMD:R_1206_3216Metric_Pad1.30x1.75mm_HandSolder -> Resistor_SMD:R_0603_1608Metric_Pad0.98x0.95mm_HandSolder; JLCPCB Part # (none) -> C114624; part number (none) -> RC0603FR-0749K9L
Connections:
- net 3.3VDC_OUT: now also C4.1, TP8.1, U1.2 (VO)
- net 5VDC_OUT: now also C10.1, C11.1, C3.1, C9.1, L1.2, R5.1, TP7.1, U1.3 (VI)
- net DC_PWR_IN: now also F2.1
- net GND: now also C1.2, C10.2, C11.2, C2.2, C3.2, C4.2, C7.2, C8.2, C9.2, D2.1, IC1.4 (GND), IC2.2 (A), R4.2, U1.1 (GND)
- net at R1.2: now also R2.1, IC1.8 (FB)
- net LM_ON_OFF: no longer names the net of R3.2
- net LM_ON_OFF: now also C1.1, IC2.1 (K), R4.1
- net LM_VIN: no longer names the net of R1.1
- net LM_VIN: now also R5.2; no longer R3.1
- new net: D2.2, D4.2 (A), F2.2, TP4.1
- new net: C14.1, R8.2
- new net BST: IC1.6 (BST), R8.1, TP5.1
- new net SW: C14.2, IC1.5 (SW), L1.1, TP6.1
- new net VIN: C2.1, C7.1, C8.1, D4.1 (K), IC1.3 (VIN), R3.1
- no-connect marks 0 -> 3
Other:
- moved on the sheet: C5, C6
